File: ESP-RGBW-3S.sch (KiCad schematic (older format))
At the start: 45 parts, among them J1 12V In, J2 PROG, J3 LED Str., J4 Temp. S., J5 Light. S., J6 PIR, J91 12V In, Q1 IRLML0040TRPBF, Q2 IRLML0040TRPBF, Q3 IRLML0040TRPBF, Q4 IRLML0040TRPBF, SW1 Flash, U2 ESP-12E, U4 DCDC_LM2596, U94 MP1584

Commit message: silk layer
Connections:
- net LED: now also R9.1; no longer R9.2
- net at D1.1 (K): now also R9.2; no longer R9.1
Changed lines of the file:
@@
 Sheet 1 1
 Title "ESP-RGBW-3S"
-Date ""
+Date "2021-05-30"
 Rev "0.4"
 Comp "Yuriy Smetana"
@@
 U 1 1 6094FB34
 P 5300 1500
-F 0 "R9" H 5370 1546 50  0000 L CNN
-F 1 "4K7" H 5370 1455 50  0000 L CNN
+F 0 "R9" H 5100 1450 50  0000 L CNN
+F 1 "4K7" H 5050 1550 50  0000 L CNN
 F 2 "Resistor_SMD:R_0805_2012Metric" V 5230 1500 50  0001 C CNN
 F 3 "~" H 5300 1500 50  0001 C CNN
 	1    5300 1500
-	1    0    0    -1
-$EndComp
-Wire Wire Line
+	-1   0    0    1
+$EndComp
+Wire Wire Line
